Commit message: car.urdf可用

File: src/apriltag_localization_simulations/urdf/car.urdf (robot description, URDF)
Before this commit: robot car, 12 links, 11 joints
Links:
- removed link body
- removed link camera_depth_optical_frame
- removed link imu
- removed link left_front_steering
- removed link left_front_wheel
- removed link left_rear_wheel
- removed link lidar
- removed link realsense
- removed link right_front_steering
- removed link right_front_wheel
- removed link right_rear_wheel
- added link camera_link; visual box size=0.05 0.05 0.05
- added link caster_back_link, mass 0.5; collision sphere radius=0.025; visual sphere radius=0.025
- added link caster_front_link, mass 0.5; collision sphere radius=0.025; visual sphere radius=0.025
- added link front_left_wheel, mass 2.5; collision cylinder length=0.02 radius=0.04; visual cylinder length=0.02 radius=0.04
- added link front_right_wheel, mass 2.5; collision cylinder length=0.02 radius=0.04; visual cylinder length=0.02 radius=0.04
- link base_link: mass None -> 5; geometry collision cylinder length=0.02 radius=0.15; visual cylinder length=0.02 radius=0.15
Joints:
- removed joint base_link_to_body
- removed joint base_link_to_left_front_steering
- removed joint base_link_to_right_front_steering
- removed joint body_to_camera_depth_optical_frame
- removed joint body_to_imu
- removed joint body_to_left_rear_wheel
- removed joint body_to_lidar
- removed joint body_to_realsense
- removed joint body_to_right_rear_wheel
- removed joint left_front_steering_to_left_front_wheel
- removed joint right_front_steering_to_right_front_wheel
- added joint camera_joint: type fixed, parent base_link, child camera_link, origin xyz=0.125 0 0.0325 rpy=0 0 0
- added joint caster_back_joint: type fixed, parent base_link, child caster_back_link, origin xyz=-0.135 0.0 0.009 rpy=-1.57079632679 0 0
- added joint caster_front_joint: type fixed, parent base_link, child caster_front_link, origin xyz=0.115 0.0 0.007 rpy=-1.57079632679 0 0
- added joint front_left_wheel_joint: type continuous, parent base_link, child front_left_wheel, origin xyz=0.0 -0.15 0.0 rpy=0 0 0, axis 0 1 0, limit effort=100 velocity=100
- added joint front_right_wheel_joint: type continuous, parent base_link, child front_right_wheel, origin xyz=0.0 0.15 0.0 rpy=0 0 0, axis 0 1 0, limit effort=100 velocity=100

File: src/apriltag_localization_simulations/urdf/my_robot.xacro (robot description, xacro)
@@ -29,11 +29,19 @@
         <material>Gazebo/Orange</material>
     </gazebo> -->
-    <gazebo reference="link_chassis">
+    <gazebo reference="base_link">
         <material>Gazebo/Orange</material>
     </gazebo>
     <gazebo reference="link_left_wheel">
+        <mu1>0.1</mu1>
+        <mu2>0.1</mu2>
+        <kp>500000.0</kp>
+        <kd>10.0</kd>
         <material>Gazebo/Blue</material>
     </gazebo>
     <gazebo reference="link_right_wheel">
+        <mu1>0.1</mu1>
+        <mu2>0.1</mu2>
+        <kp>500000.0</kp>
+        <kd>10.0</kd>
         <material>Gazebo/Blue</material>
     </gazebo>
@@ -42,6 +50,6 @@
             <alwaysOn>true</alwaysOn>
             <updateRate>50.0</updateRate>
-            <leftJoint>car_base_front_left_wheel</leftJoint>
-            <rightJoint>car_base_front_right_wheel</rightJoint>
+            <leftJoint>joint_left_wheel</leftJoint>
+            <rightJoint>joint_right_wheel</rightJoint>
             <wheelSeparation>1.0</wheelSeparation>
             <wheelDiameter>0.5</wheelDiameter>
@@ -58,51 +66,38 @@
     </gazebo> -->
     <gazebo reference="camera_link">
-    <material>Gazebo/Green</material>
-    <sensor type="camera" name="camera1">
-      <update_rate>30.0</update_rate>
-      <camera name="head">
-        <horizontal_fov>1.3962634</horizontal_fov>
-        <image>
-          <width>800</width>
-          <height>800</height>
-          <format>R8G8B8</format>
-        </image>
-        <clip>
-          <near>0.02</near>
-          <far>300</far>
-        </clip>
-      </camera>
-      <plugin name="camera_controller" filename="libgazebo_ros_camera.so">
-        <alwaysOn>true</alwaysOn>
-        <updateRate>0.0</updateRate>
-        <cameraName>my_robot/camera1</cameraName>
-        <imageTopicName>image_raw</imageTopicName>
-        <cameraInfoTopicName>camera_info</cameraInfoTopicName>
-        <frameName>camera</frameName>
-        <hackBaseline>0.07</hackBaseline>
-        <distortionK1>0.0</distortionK1>
-        <distortionK2>0.0</distortionK2>
-        <distortionK3>0.0</distortionK3>
-        <distortionT1>0.0</distortionT1>
-        <distortionT2>0.0</distortionT2>
-      </plugin>
-    </sensor>
-  </gazebo>
+        <material>Gazebo/Green</material>
+        <sensor type="camera" name="camera1">
+            <update_rate>30.0</update_rate>
+            <camera name="head">
+                <horizontal_fov>1.3962634</horizontal_fov>
+                <image>
+                    <width>800</width>
+                    <height>800</height>
+                    <format>R8G8B8</format>
+                </image>
+                <clip>
+                    <near>0.02</near>
+                    <far>300</far>
+                </clip>
+            </camera>
+            <plugin name="camera_controller" filename="libgazebo_ros_camera.so">
+                <alwaysOn>true</alwaysOn>
+                <updateRate>0.0</updateRate>
+                <cameraName>my_robot/camera1</cameraName>
+                <imageTopicName>image_raw</imageTopicName>
+                <cameraInfoTopicName>camera_info</cameraInfoTopicName>
+                <frameName>camera</frameName>
+                <hackBaseline>0.07</hackBaseline>
+                <distortionK1>0.0</distortionK1>
+                <distortionK2>0.0</distortionK2>
+                <distortionK3>0.0</distortionK3>
+                <distortionT1>0.0</distortionT1>
+                <distortionT2>0.0</distortionT2>
+            </plugin>
+        </sensor>
+    </gazebo>
     <link name="base_link">
-        <visual>
-            <geometry>
-                <box size =".001 .001 .001"/>
-            </geometry>
-            <origin rpy="0 0 0" xyz="0 0 0"/>
-        </visual>
-    </link>
-    <joint name="base_link_car" type="fixed">
-        <origin xyz="0.0 0.0 0.0" rpy="0.0 0.0 0.0"/>
-        <parent link="base_link"/>
-        <child link="link_chassis"/>
-    </joint>
-    <link name="link_chassis">
         <!-- pose and inertial -->
-        <pose>0 0 1 0 0 0</pose>
+        <pose>0 0 0.4 0 0 0</pose>
         <inertial>
             <mass value="15.0"/>
@@ -110,5 +105,5 @@
             <inertia ixx="0.12" ixy="0" ixz="0" iyy="0.1" iyz="0" izz="0.1" />
         </inertial>
-        <collision name="collision_chassis">
+        <collision name="collision_base">
             <geometry>
                 <box size="1 0.8 0.4"/>
@@ -132,4 +127,6 @@
                         <mu>0</mu>
                         <mu2>0</mu2>
+                        <kp>500000.0</kp>
+                        <kd>10.0</kd>
                         <slip1>1.0</slip1>
                         <slip2>1.0</slip2>
@@ -146,11 +143,9 @@
     </link>
     <!--   Joint for chassis  -->
-    <!-- <joint name="joint_chassis" type="continuous">
+    <!-- <joint name="joint_base" type="fixed">
         <origin rpy="0 0 0" xyz="0 0 0.4"/>
-        <child link="link_chassis" />
-        <parent link="base_link"/>
-        <axis rpy="0 0 0" xyz="0 1 0"/>
-        <limit effort="10000" velocity="1000"/>
-        <joint_properties damping="1.0" friction="1.0" />
+        <axis rpy="0 0 0" xyz="0 0 0"/>
+        <limit effort="10000" velocity="1000"/>
+        <joint_properties damping="1.0" friction="0.5" />
     </joint> -->
     <!-- Create camera link -->
@@ -178,12 +173,12 @@
         <origin rpy="0 0 0" xyz="0.5 0 0.3"/>
         <child link="camera_link" />
-        <parent link="link_chassis"/>
+        <parent link="base_link"/>
         <axis rpy="0 0 0" xyz="0 1 0"/>
         <limit effort="10000" velocity="1000"/>
-        <joint_properties damping="1.0" friction="1.0" />
+        <joint_properties damping="1.0" friction="0.5" />
     </joint>
     <!-- Create wheel right -->
     <link name="link_right_wheel">
-         <inertial>
+        <inertial>
             <origin xyz="0 0 0" rpy="0 1.5707 1.5707"/>
             <mass value="5"/>
@@ -207,12 +202,12 @@
         <origin rpy="0 0 0" xyz="0.333838 -0.6 -0.15"/>
         <child link="link_right_wheel" />
-        <parent link="link_chassis"/>
+        <parent link="base_link"/>
         <axis xyz="0 1 0" rpy="0 0 0"/>
         <limit effort="10000" velocity="1000"/>
-        <joint_properties damping="1.0" friction="1.0"/>
+        <joint_properties damping="1.0" friction="0.5"/>
     </joint>
     <!-- Left Wheel link -->
     <link name="link_left_wheel">
-         <inertial>
+        <inertial>
             <origin xyz="0 0 0" rpy="0 1.5707 1.5707"/>
             <mass value="5"/>
@@ -236,8 +231,8 @@
         <origin rpy="0 0 0" xyz="0.333838 0.6 -0.15"/>
         <child link="link_left_wheel" />
-        <parent link="link_chassis"/>
+        <parent link="base_link"/>
         <axis xyz="0 1 0" rpy="0 0 0"/>
         <limit effort="10000" velocity="1000"/>
-        <joint_properties damping="1.0" friction="1.0"/>
+        <joint_properties damping="1.0" friction="0.5"/>
     </joint>
 </robot>

File: src/apriltag_localization_simulations/urdf/robot.xacro (robot description, xacro)
@@ -1,47 +1,47 @@
 <?xml version="1.0"?>
-<robot name="robot"
+<robot name="my_robot"
     xmlns:xacro="http://www.ros.org/wiki/xacro">
-<gazebo reference="chassis">
-    <material>Gazebo/Orange</material>
-  </gazebo>
-  <gazebo reference="left_wheel">
-    <material>Gazebo/Blue</material>
-  </gazebo>
-  <gazebo reference="right_wheel">
-    <material>Gazebo/Blue</material>
-  </gazebo>sudo
-<gazebo reference="camera">
-    <material>Gazebo/Green</material>
-    <sensor type="camera" name="camera1">
-      <update_rate>30.0</update_rate>
-      <camera name="head">
-        <horizontal_fov>1.3962634</horizontal_fov>
-        <image>
-          <width>800</width>
-          <height>800</height>
-          <format>R8G8B8</format>
-        </image>
-        <clip>
-          <near>0.02</near>
-          <far>300</far>
-        </clip>
-      </camera>
-      <plugin name="camera_controller" filename="libgazebo_ros_camera.so">
-        <alwaysOn>true</alwaysOn>
-        <updateRate>0.0</updateRate>
-        <cameraName>robot/camera1</cameraName>
-        <imageTopicName>image_raw</imageTopicName>
-        <cameraInfoTopicName>camera_info</cameraInfoTopicName>
-        <frameName>camera</frameName>
-        <hackBaseline>0.07</hackBaseline>
-        <distortionK1>0.0</distortionK1>
-        <distortionK2>0.0</distortionK2>
-        <distortionK3>0.0</distortionK3>
-        <distortionT1>0.0</distortionT1>
-        <distortionT2>0.0</distortionT2>
-      </plugin>
-    </sensor>
-  </gazebo>
-    <link name='chassis'>
+    <gazebo reference="base_link">
+        <material>Gazebo/Orange</material>
+    </gazebo>
+    <gazebo reference="left_wheel">
+        <material>Gazebo/Blue</material>
+    </gazebo>
+    <gazebo reference="right_wheel">
+        <material>Gazebo/Blue</material>
+    </gazebo>sudo
+    <gazebo reference="camera_link">
+        <material>Gazebo/Green</material>
+        <sensor type="camera" name="camera1">
+            <update_rate>30.0</update_rate>
+            <camera name="head">
+                <horizontal_fov>1.3962634</horizontal_fov>
+                <image>
+                    <width>800</width>
+                    <height>800</height>
+                    <format>R8G8B8</format>
+                </image>
+                <clip>
+                    <near>0.02</near>
+                    <far>300</far>
+                </clip>
+            </camera>
+            <plugin name="camera_controller" filename="libgazebo_ros_camera.so">
+                <alwaysOn>true</alwaysOn>
+                <updateRate>0.0</updateRate>
+                <cameraName>my_robot/camera1</cameraName>
+                <imageTopicName>image_raw</imageTopicName>
+                <cameraInfoTopicName>camera_info</cameraInfoTopicName>
+                <frameName>camera</frameName>
+                <hackBaseline>0.07</hackBaseline>
+                <distortionK1>0.0</distortionK1>
+                <distortionK2>0.0</distortionK2>
+                <distortionK3>0.0</distortionK3>
+                <distortionT1>0.0</distortionT1>
+                <distortionT2>0.0</distortionT2>
+            </plugin>
+        </sensor>
+    </gazebo>
+    <link name='base_link'>
         <pose>0 0 0.1 0 0 0</pose>
         <inertial>
@@ -55,5 +55,5 @@
             </geometry>
         </collision>
-        <visual name='chassis_visual'>
+        <visual name='base_link_visual'>
             <origin xyz="0 0 0" rpy=" 0 0 0"/>
             <geometry>
@@ -106,27 +106,24 @@
         </visual>
     </link>
-<link name="right_wheel">
-    <!--origin xyz="0.1 0.13 0.1" rpy="0 1.5707 1.5707"/-->
-    <collision name="collision">
-      <origin xyz="0 0 0" rpy="0 1.5707 1.5707"/>
-      <geometry>
-        <cylinder radius="0.1" length="0.05"/>
-      </geometry>
-    </collision>
-    <visual name="right_wheel_visual">
-      <origin xyz="0 0 0" rpy="0 1.5707 1.5707"/>
-      <geometry>
-        <cylinder radius="0.1" length="0.05"/>
-      </geometry>
-    </visual>
-    <inertial>
-      <origin xyz="0 0 0" rpy="0 1.5707 1.5707"/>
-      <mass value="5"/>
-      <inertia
-        ixx=".1" ixy="0.0" ixz="0.0"
-        iyy=".1" iyz="0.0"
-        izz=".1"/>
-    </inertial>
-  </link>
+    <link name="right_wheel">
+        <!--origin xyz="0.1 0.13 0.1" rpy="0 1.5707 1.5707"/-->
+        <collision name="collision">
+            <origin xyz="0 0 0" rpy="0 1.5707 1.5707"/>
+            <geometry>
+                <cylinder radius="0.1" length="0.05"/>
+            </geometry>
+        </collision>
+        <visual name="right_wheel_visual">
+            <origin xyz="0 0 0" rpy="0 1.5707 1.5707"/>
+            <geometry>
+                <cylinder radius="0.1" length="0.05"/>
+            </geometry>
+        </visual>
+        <inertial>
+            <origin xyz="0 0 0" rpy="0 1.5707 1.5707"/>
+            <mass value="5"/>
+            <inertia ixx=".1" ixy="0.0" ixz="0.0" iyy=".1" iyz="0.0" izz=".1"/>
+        </inertial>
+    </link>
     <link name="left_wheel">
         <!--origin xyz="0.1 0.13 0.1" rpy="0 1.5707 1.5707"/-->
@@ -153,5 +150,5 @@
         <!--origin xyz="0.1 0.13 0" rpy="0 1.5707 1.5707"/-->
         <child link="left_wheel"/>
-        <parent link="chassis"/>
+        <parent link="base_link"/>
         <axis xyz="0 1 0" rpy="0 0 0"/>
         <limit effort="10000" velocity="1000"/>
@@ -161,35 +158,35 @@
         <origin xyz="0 -0.15 0" rpy="0 0 0"/>
         <child link="right_wheel"/>
-        <parent link="chassis"/>
+        <parent link="base_link"/>
         <axis xyz="0 1 0" rpy="0 0 0"/>
         <limit effort="10000" velocity="1000"/>
         <joint_properties damping="1.0" friction="1.0"/>
     </joint>
-    <link name="camera">
-    <collision>
-      <origin xyz="0 0 0" rpy="0 0 0"/>
-      <geometry>
-        <box size="0.1 0.1 0.1"/>
-      </geometry>
-    </collision>
-    <visual>
-      <origin xyz="0 0 0" rpy="0 0 0"/>
-      <geometry>
-        <box size="0.1 0.1 0.1"/>
-      </geometry>
-      <material name="green"/>
-    </visual>
-    <inertial>
-      <mass value="1.0" />
-      <origin xyz="0 0 0" rpy="0 0 0"/>
-      <box_inertia m="1.0" x="0.1" y="0.1" z="0.1" />
-      <inertia ixx="1e-6" ixy="0" ixz="0" iyy="1e-6" iyz="0" izz="1e-6" />
-    </inertial>
-  </link>
-  <joint name="camera_joint" type="fixed">
-    <axis xyz="0 1 0" />
-    <origin xyz=".2 0 0" rpy="0 0 0"/>
-    <parent link="chassis"/>
-    <child link="camera"/>
-  </joint>
+    <link name="camera_link">
+        <collision>
+            <origin xyz="0 0 0" rpy="0 0 0"/>
+            <geometry>
+                <box size="0.1 0.1 0.1"/>
+            </geometry>
+        </collision>
+        <visual>
+            <origin xyz="0 0 0" rpy="0 0 0"/>
+            <geometry>
+                <box size="0.1 0.1 0.1"/>
+            </geometry>
+            <material name="green"/>
+        </visual>
+        <inertial>
+            <mass value="1.0" />
+            <origin xyz="0 0 0" rpy="0 0 0"/>
+            <box_inertia m="1.0" x="0.1" y="0.1" z="0.1" />
+            <inertia ixx="1e-6" ixy="0" ixz="0" iyy="1e-6" iyz="0" izz="1e-6" />
+        </inertial>
+    </link>
+    <joint name="camera_joint" type="fixed">
+        <axis xyz="0 1 0" />
+        <origin xyz="0 0 .3" rpy="0 0 0"/>
+        <parent link="base_link"/>
+        <child link="camera_link"/>
+    </joint>
 </robot>
